File: remote/Hardware/remote.brd (EAGLE design)
At the start: 54 x 70.5 mm, 30 parts, among them IC1 TINY13-20PU

Commit message: Naprawa Plytki pilota, gotowe do termotransferu
Parts:
- moved R6 9.76 mm to (47.5, 54.9)
- moved SCRL_DOWN 7.00 mm to (52.0, 37.0)
- moved SCRL_OK 7.00 mm to (52.0, 47.0)
- moved SCRL_UP 7.00 mm to (52.0, 57.0)
- moved X1 6.59 mm to (4.77, 16.6), turned to 90 degrees
- moved R7 6.47 mm to (44.5, 47.7)
- moved R8 3.56 mm to (47.0, 39.7)
- moved R2 3.28 mm to (16.8, 62.1)
Routing:
- net GND: track 159.7 -> 172.9 mm
- net VCC: track 251.3 -> 257.6 mm
- net N$12: track 17.4 -> 12.4 mm
- net N$5: track 17.1 -> 13.8 mm
- net N$6: track 34.2 -> 37.0 mm
- net N$8: track 10.3 -> 12.9 mm
- net N$7: track 11.4 -> 10.3 mm
- net N$9: track 19.5 -> 18.6 mm
Other:
- board text added: "FIRMWARE"
- board text added: "IR_Mouse"
- board text added: "Remote"
- board text removed: "FIRMWARE UPGRADE"
